File: CheapMesh_KiCad/CheapMesh.kicad_pcb (KiCad board)
At the start: 2 copper layers, 34.8 x 67.3 mm, 25 parts, among them J1 Conn_01x02_Pin, J2 Conn_01x09_Pin, J3 USB_A, J4 USB_C, J5 Conn_Coaxial, Q1 UMH3N, U1 L78L33, U2 HT-CT62, U3 AP2112K-3.3

Commit message: update version
Other:
- board text added: "Cheap/\/\esh by PaulHausK & joyel24 v1.4.4"
- board text removed: "Cheap/\/\esh by PaulHausK & joyel24 v1.4.3"
Changed lines of the file:
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@@
 		)
 	)
-	(gr_text "Cheap/\\/\\esh\nby PaulHausK\n& joyel24\nv1.4.3\n"
+	(gr_text "Cheap/\\/\\esh\nby PaulHausK\n& joyel24\nv1.4.4\n"
 		(at 33.75 149.75 270)
 		(layer "F.SilkS")
